Commit message: Stabilized landing on dynamic AR tag by bottm camera.

File: src/simulation/car/car_description/sdf/macros.xacro (robot description, xacro)
@@ -33,5 +33,5 @@
 <macro name="wheel" params="lr tY">
  <link name="${lr}_wheel">
-   <pose>${wheelPos} ${tY*wheelWidth/2+tY*chassisWidth/2} ${wheelRadius} 0 ${PI/2} ${PI/2}</pose>
+   <pose>${wheelPos} ${tY*wheelWidth/2+tY*chassisWidth/2} ${wheelRadius-chassisHeight/2} 0 ${PI/2} ${PI/2}</pose>
    <collision name="${lr}_wheel_collision">
     <geometry>

File: src/simulation/car/car_description/sdf/model.sdf.xacro (robot description, xacro)
@@ -7,6 +7,4 @@
     <xacro:property name="chassisWidth" value="0.5"/>
     <xacro:property name="chassisMass" value="50"/>
-    <xacro:property name="casterRadius" value="0.03"/>
-    <xacro:property name="casterMass" value="5"/>
     <xacro:property name="wheelWidth" value="0.05"/>
     <xacro:property name="wheelRadius" value="0.08"/>
@@ -14,4 +12,6 @@
     <xacro:property name="wheelMass" value="5"/>
     <xacro:property name="wheelDamping" value="1"/>
+    <xacro:property name="casterRadius" value="${wheelRadius}"/>
+    <xacro:property name="casterMass" value="5"/>
     <xacro:property name="cameraSize" value="0.05"/>
     <xacro:property name="cameraMass" value="0.1"/>
