Commit message: Minor updates to the project

File: src/simulation/car/car_description/sdf/model.sdf.xacro (robot description, xacro)
@@ -3,5 +3,5 @@
   <model name="Car" xmlns:xacro="http://www.ros.org/wiki/xacro">
     <xacro:property name="PI" value="3.1415926535897931"/>
-    <xacro:property name="chassisHeight" value="0.1"/>
+    <xacro:property name="chassisHeight" value="0.5"/>
     <xacro:property name="chassisLength" value="0.5"/>
     <xacro:property name="chassisWidth" value="0.5"/>

Commit message: Resolved conflicts.

File: src/simulation/car/car_description/sdf/model.sdf.xacro (robot description, xacro)
@@ -3,5 +3,5 @@
   <model name="Car" xmlns:xacro="http://www.ros.org/wiki/xacro">
     <xacro:property name="PI" value="3.1415926535897931"/>
-    <xacro:property name="chassisHeight" value="0.5"/>
+    <xacro:property name="chassisHeight" value="0.1"/>
     <xacro:property name="chassisLength" value="0.5"/>
     <xacro:property name="chassisWidth" value="0.5"/>
